File: bottle-light.brd (EAGLE design)
At the start: 88 x 88 mm, 51 parts, among them IC1 STM32F334K8T, IC2 LF33, X1 78127-1128, X2 61300411121, X3 SWD, X4 UJ2-MIBH-4-SMT-TR

Commit message: Update README | added images of schematic, board and 3D view
Parts:
- added U$1: (no value), frames:A4L-LOC
Changed lines of the file:
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@@
 <drawing>
 <settings>
-<setting alwaysvectorfont="yes"/>
+<setting alwaysvectorfont="no"/>
 <setting keepoldvectorfont="yes"/>
 <setting verticaltext="up"/>
 </settings>
-<grid distance="1" unitdist="mm" unit="mm" style="lines" multiple="1" display="yes" altdistance="0.25" altunitdist="mm" altunit="mm"/>
+<grid distance="5" unitdist="mm" unit="mm" style="lines" multiple="1" display="yes" altdistance="0.25" altunitdist="mm" altunit="mm"/>
 <layers>
 <layer number="1" name="Top" color="4" fill="1" visible="yes" active="yes"/>
@@
 <layer number="46" name="Milling" color="3" fill="1" visible="no" active="yes"/>
 <layer number="47" name="Measures" color="7" fill="1" visible="no" active="yes"/>
-<layer number="48" name="Document" color="7" fill="1" visible="no" active="yes"/>
+<layer number="48" name="Document" color="7" fill="1" visible="yes" active="yes"/>
 <layer number="49" name="Reference" color="7" fill="1" visible="no" active="yes"/>
 <layer number="50" name="dxf" color="7" fill="1" visible="no" active="no"/>
@@
 <attribute name="VALUE" x="61" y="65.5999" size="0.02" layer="28" rot="MR270"/>
 </element>
+<element name="U$1" library="frames" library_urn="urn:adsk.eagle:library:229" package="A4L-LOC" value="" x="-85" y="-45" smashed="yes">
+<attribute name="DRAWING_NAME" x="132.17" y="-29.76" size="2.54" layer="48" font="vector"/>
+<attribute name="LAST_DATE_TIME" x="132.17" y="-34.84" size="2.286" layer="48" font="vector"/>
+</element>
 </elements>

Commit message: changed some footprint drawings
Parts:
- flipped X2 to the bottom, turned to 180 degrees
Other:
- outline, holes or cut-outs redrawn
- board text added: "5V"
- board text added: "BottleLight v0.2.8 04.07.2019 by HansAchterbahn MIT Licence https://github.com/ HansAchterbahn/bottle-light"
- board text added: "CLK"
- board text added: "GND"
- board text added: "MOSI"
- board text removed: "BottleLight v0.2.7 27.06.2019 HansAchterbahn MIT Licence"
